Commit message: updated urdf to reorient imu

File: pi_mapping/urdf/base_descr.urdf.xacro (robot description, xacro)
@@ -12,5 +12,5 @@
 	<xacro:arg name="cam_yaw" default="0.0" />
 	<xacro:arg name="has_imu" default="false" />
-	<xacro:include filename="$(find remote_rtabmap)/urdf/include/base_macro.urdf.xacro" />
+	<xacro:include filename="$(find pi_mapping)/urdf/include/base_macro.urdf.xacro" />
 	<link name="$(arg parent_frame)" />
 	<xacro:base camera_name="$(arg camera_name)" parent="$(arg parent_frame)"

File: pi_mapping/urdf/depthai_descr.urdf.xacro (robot description, xacro)
@@ -12,5 +12,5 @@
 	<xacro:arg name="cam_yaw" default="0.0" />
 	<xacro:arg name="rs_compat" default="false" />
-	<xacro:include filename="$(find remote_rtabmap)/urdf/include/depthai_macro.urdf.xacro" />
+	<xacro:include filename="$(find pi_mapping)/urdf/include/depthai_macro.urdf.xacro" />
 	<link name="$(arg parent_frame)" />
 	<xacro:depthai_camera camera_name="$(arg camera_name)" parent="$(arg parent_frame)"

File: pi_mapping/urdf/include/base_macro.urdf.xacro (robot description, xacro)
@@ -65,6 +65,6 @@
 			<xacro:property name="imu_offset_y" value="-0.015" />
 			<xacro:property name="imu_offset_z" value="-0.013662" />
-			<xacro:property name="imu_r" value="0.0" />
-			<xacro:property name="imu_p" value="${M_PI/2.0}" />
+			<xacro:property name="imu_r" value="${M_PI/2.0}" />
+			<xacro:property name="imu_p" value="0.0" />
 			<xacro:property name="imu_y" value="0.0" />
 		</xacro:if>

File: pi_mapping/urdf/include/depthai_macro.urdf.xacro (robot description, xacro)
@@ -6,5 +6,5 @@
                                            cam_pos_x cam_pos_y cam_pos_z
                                            cam_roll cam_pitch cam_yaw r:=0.8 g:=0.8 b:=0.8 a:=0.8 simulation:=false rs_compat:=false">
-		<xacro:include filename="$(find remote_rtabmap)/urdf/include/base_macro.urdf.xacro" />
+	<xacro:include filename="$(find pi_mapping)/urdf/include/base_macro.urdf.xacro" />
 		<xacro:property name="M_PI" value="3.1415926535897931" />
 		<xacro:property name="model" value="${camera_model}" />
